File: pcb/print.kicad_pcb (KiCad board)
At the start: 2 copper layers, 0 parts

Commit message: First production update.
Parts:
- added C1: 100nF, Capacitor_SMD:C_0402_1005Metric, F.Cu at (153.5, 101.8)
- added C2: 100nF, Capacitor_SMD:C_0402_1005Metric, F.Cu at (153.6, 84.3)
- added C3: 100nF, Capacitor_SMD:C_0402_1005Metric, F.Cu at (155.0, 106.6)
- added C4: 4.7nF/1kV, Capacitor_SMD:C_0402_1005Metric, F.Cu at (149.7, 113.8)
- added D1: PRTR5V0U2X, Package_TO_SOT_SMD:SOT-143, F.Cu at (147.0, 115.9)
- added D3: CPU, Diode_SMD:D_0603_1608Metric, F.Cu at (147.4, 83.3)
- added J1: USB_C_Receptacle_USB2.0_16P, Connector_USB:USB_C_Receptacle_GCT_USB4105-xx-A_16P_TopMnt_Horizontal, F.Cu at (150.6, 122.4)
- added J2: WS2812, Connector_PinHeader_2.54mm:PinHeader_1x03_P2.54mm_Vertical, F.Cu at (153.0, 80.3)
- added R1: 5K1, Resistor_SMD:R_0402_1005Metric, F.Cu at (152.3, 116.6)
- added R2: 5K1, Resistor_SMD:R_0402_1005Metric, F.Cu at (149.3, 116.6)
- added R3: 10K0, Resistor_SMD:R_0402_1005Metric, F.Cu at (155.0, 103.7)
- added R4: 1M0, Resistor_SMD:R_0402_1005Metric, F.Cu at (149.8, 114.9)
- added R6: 4K7, Resistor_SMD:R_0402_1005Metric, F.Cu at (149.5, 83.8)
- added SW1: Cycle, Button_Switch_THT:SW_PUSH_6mm_H4.3mm, F.Cu at (148.3, 99.6)
- added U1: ATtiny85-20S, Package_SO:SOIC-8_5.3x5.3mm_P1.27mm, F.Cu at (150.5, 87.9)
- added U2: CH340C, Package_SO:SOIC-16_3.9x9.9mm_P1.27mm, F.Cu at (150.6, 107.7)
Routing:
- net VBUS: track 0.00 -> 85.6 mm, vias 0 -> 2
- net /~{Reset} : track 0.00 -> 28.8 mm, vias 0 -> 2
- net /USB_D_N: track 0.00 -> 22.8 mm, vias 0 -> 2
- net /TX_D_P: track 0.00 -> 21.4 mm
- net /RX_D_P: track 0.00 -> 21.3 mm
- net /USB_D_P: track 0.00 -> 20.5 mm, vias 0 -> 2
- net Net-(U1-XTAL1/PB3): track 0.00 -> 16.3 mm
- net /LED_DATA_P: track 0.00 -> 10.1 mm
- net Net-(U1-XTAL2/PB4): track 0.00 -> 6.40 mm
- net GND: track 0.00 -> 2.72 mm, vias 0 -> 15
- net Net-(D1-GND): track 0.00 -> 2.65 mm
- net Net-(U2-~{DTR}): track 0.00 -> 1.95 mm
- net Net-(J1-CC2): track 0.00 -> 1.68 mm
- net Net-(J1-CC1): track 0.00 -> 1.68 mm
- net Net-(D3-A): track 0.00 -> 1.33 mm
- added copper zone on B.Cu, net GND
- added copper zone on F.Cu, net GND
Other:
- board outline added: 11.2 x 46.4 mm
- board text added: "Do Not Disturb Indicator v1.0.0 - 00.25.0029 MonkeyEnterprise"
