File: pcb/print.kicad_sch (KiCad schematic)
At the start: 22 parts, among them J1 USB_C_Receptacle_USB2.0_16P, J2 WS2812, SW1 Cycle, U1 FT232RL, U2 ATtiny85-20S

Commit message: pcb v1.1.0 update
Parts:
- removed C1, C4: 100nF, Capacitor_SMD:C_0402_1005Metric, symbol Device:C_Small
- removed D1, D2, D3, D4: WS2812B, LED_SMD:LED_WS2812B_PLCC4_5.0x5.0mm_P3.2mm, symbol LED:WS2812B
- removed J2: WS2812, Connector_PinHeader_2.54mm:PinHeader_1x03_P2.54mm_Vertical, symbol Connector:Conn_01x03_Pin
- removed U1: FT232RL, Package_SO:SSOP-28_5.3x10.2mm_P0.65mm, symbol Interface_USB:FT232RL
- added C10, C11, C12, C13, C6, C7, C8, C9: 100nF, Capacitor_SMD:C_0402_1005Metric, symbol Device:C_Small
- added D1: PRTR5V0U2X, Package_TO_SOT_SMD:SOT-143, symbol Power_Protection:PRTR5V0U2X
- added D10, D3, D4, D5, D6, D7, D8, D9: WS2812B, Lib_WS2812B:LED_WS2812B_PLCC4_5.0x5.0mm_P3.2mm, symbol Lib_WS2812B:WS2812B
- added R4, R5: 1K0, Resistor_SMD:R_0402_1005Metric, symbol Device:R_Small
- added R8: 1M0, Resistor_SMD:R_0402_1005Metric, symbol Device:R_Small
- added U2: CH340C, Package_SO:SOIC-16_3.9x9.9mm_P1.27mm, symbol Interface_USB:CH340C
- C5: value 100nF -> 4.7nF/1kV; LCSC C1525 -> C1538
- R1: value 4K7 -> 1K0
- renumbered C7 to C1, C6 to C4, D5 to D2, R5 to R6, R4 to R7, U2 to U1
Connections:
- net +3.3V is gone; now on net VBUS: C2.1
- net GND: now also C10.2, C11.2, C12.2, C13.2, C6.2, C7.2, C8.2, C9.2, D10.3 (VSS), D3.3 (VSS), D4.3 (VSS), D5.3 (VSS), D6.3 (VSS), D7.3 (VSS), D8.3 (VSS), D9.3 (VSS), R8.2, U2.1 (GND)
- net LED_DATA_P: now also D3.4 (DIN), R5.2; no longer R1.1, U1.7 (PB2)
- net VBUS: now also C10.1, C11.1, C12.1, C13.1, C6.1, C7.1, C8.1, C9.1, D1.4 (VCC), D10.1 (VDD), D3.1 (VDD), D4.1 (VDD), D5.1 (VDD), D6.1 (VDD), D7.1 (VDD), D8.1 (VDD), D9.1 (VDD), U2.16 (VCC); no longer C3.1, C5.1
- net TX_D_P: now reaches R1.2
- net TX_D_P: now also U2.3 (RXD)
- net at C4.1: now also U2.13 (~{DTR})
- net RX: no longer names the net of U1.6 (PB1)
- net RX: now also R4.1
- net TX: no longer names the net of U1.5 (AREF/PB0)
- net TX: now also R1.1
- net USB_N renamed USB_D_N
- net USB_D_N: now also D1.3 (I/O2), U2.6 (UD-)
- net USB_P renamed USB_D_P
- net USB_D_P: now also D1.2 (I/O1), U2.5 (UD+)
- new net: D6.2 (DOUT), D7.4 (DIN)
- new net: D5.2 (DOUT), D6.4 (DIN)
- new net: C3.1, U2.4 (V3)
- new net: C5.1, D1.1 (GND), R8.1
- new net: R5.1, U1.7 (PB2)
- new net: D8.2 (DOUT), D9.4 (DIN)
- new net: D7.2 (DOUT), D8.4 (DIN)
- new net: D4.2 (DOUT), D5.4 (DIN)
- new net: D3.2 (DOUT), D4.4 (DIN)
- new net: D10.4 (DIN), D9.2 (DOUT)
- new net RX_D_P: R4.2, U2.2 (TXD)
- no-connect marks 15 -> 9
Other:
- note added: "ESD Protection"
- moved on the sheet: C2, C4, J1, R7
